File: PCB/HyprBoard.kicad_sch (KiCad schematic)
At the start: 33 parts, among them J1 USB_C_Receptacle_USB2.0_14P, J2 Conn_01x20_Pin, J3 Conn_01x20_Pin, J4 Conn_01x03_Pin, SW1 SW_Push, U1 RP2040, U2 NCP1117-3.3_SOT223, U3 W25Q128JVS, Y1 12 MHz

Commit message: Rage quit tryna route the pcb, please pray for me.. thanks!
Parts:
- removed U2: NCP1117-3.3_SOT223, Package_TO_SOT_SMD:SOT-223-3_TabPin2, symbol Regulator_Linear:NCP1117-3.3_SOT223
- added D1: LED, LED_SMD:LED_0402_1005Metric, symbol Device:LED
- added R8: 0.22K, Resistor_SMD:R_0402_1005Metric, symbol Device:R
- added U2: MCP1700x-330xxTT, Package_TO_SOT_SMD:SOT-23, symbol Regulator_Linear:MCP1700x-330xxTT
- U3: value W25Q128JVS -> W25Q16JVZPIQ TR; footprint Package_SO:SOIC-8_5.3x5.3mm_P1.27mm -> Package_SON:Winbond_USON-8-1EP_3x2mm_P0.5mm_EP0.2x1.6mm
Connections:
- net +3V3: now also U2.2 (VO)
- net GND: now also D1.1 (K), U2.1 (GND)
- net VBUS: now also U2.3 (VI)
- net at U1.37 (GPIO25): now also R8.1
- new net: D1.2 (A), R8.2
- no-connect marks 1 -> 0
